File: Git Tutorial 3.kicad_sch (KiCad schematic)
At the start: 0 parts

Commit message: schematic updated
Parts:
- added BT1: Battery_Cell, symbol Device:Battery_Cell
- added D1: LED, symbol Device:LED
- added R1: R_Small, symbol Device:R_Small
Connections:
- new net: BT1.1 (+), R1.2
- new net: BT1.2 (-), D1.1 (K)
- new net: D1.2 (A), R1.1
